Commit message: Adicionando a clase do Grasp-e

File: ros_ws/src/graspe_description/urdf/robot.urdf (robot description, URDF)
Before this commit: robot graspe, 4 links, 3 joints
Links:
- removed link end_effector
- removed link linear_arm
- removed link rotating_arm
- added link endfactor_link; visual box size=0.16 0.1 0.1
- added link extendarm_link; visual cylinder length=0.2 radius=0.04
- added link head_link; visual box size=0.1 0.1 0.1
- added link pillar_link; visual cylinder length=0.5 radius=0.05
- added link shoulder_link; visual box size=0.14 0.1 0.1
- added link upperarm_link; visual box size=0.16 0.1 0.1
- link base_link: geometry visual cylinder length=0.1 radius=0.2
Joints:
- removed joint base_to_rotating_arm
- removed joint linear_arm_to_end_effector
- removed joint rotating_arm_to_linear_arm
- added joint base_pilar_joint: type fixed, parent base_link, child pillar_link, origin xyz=0.0 0.0 0.0 rpy=0.0 0.0 0.0, axis 0.0 0.0 0.0, limit lower=0.0 upper=0.0 effort=0.0 velocity=0.0
