Commit message: Controler semi-fixed

File: ros_ws/src/graspe_description/urdf/graspe.xacro (robot description, xacro)
@@ -1,8 +1,9 @@
 <?xml version="1.0" ?>
 <robot name="graspe" xmlns:xacro="http://www.ros.org/wiki/xacro">
-<xacro:arg name="is_ignition" default="true"/>
 <xacro:include filename="$(find graspe_description)/urdf/materials.xacro" />
 <xacro:include filename="$(find graspe_description)/urdf/graspe.trans" />
 <xacro:include filename="$(find graspe_description)/urdf/graspe.gazebo" />
+<xacro:include filename="$(find graspe_description)/urdf/graspe_joints_limits.xacro" />
+<xacro:include filename="$(find graspe_description)/urdf/graspe_gazebo_control.xacro" />
 <!-- Theta1 -->
 <xacro:property name="ajuste1" value="0.04"/>
@@ -55,9 +56,10 @@
   </collision>
 </link>
-<joint name="theta1" type="continuous">
+<joint name="theta1" type="revolute">
   <origin xyz="0.0 0.0 0.053" rpy="0 0 0"/>
   <parent link="base_link"/>
   <child link="revolution_link_1"/>
   <axis xyz="0.0 0.0 1.0"/>
+  <limit upper="${theta1_max}" lower="${theta1_min}" effort="${effort_max}" velocity="${velocity_max}"/>
 </joint>
 <!-- Fixed jointJoint -->
@@ -113,5 +115,5 @@
   <child link="revolution2_link_1"/>
   <axis xyz="0.0 -1.0 0.0"/>
-  <limit upper="0.785398" lower="-0.785398" effort="100" velocity="100"/>
+  <limit upper="${theta2_max}" lower="${theta2_min}" effort="${effort_max}" velocity="${velocity_max}"/>
 </joint>
 <!-- d3 -->
@@ -141,5 +143,5 @@
   <child link="slider_link_1"/>
   <axis xyz="0.0 0.0 1.0"/>
-  <limit upper="0.0" lower="-0.026" effort="100" velocity="100"/>
+  <limit upper="${d3_max}" lower="${d3_min}" effort="${effort_max}" velocity="${velocity_max}"/>
 </joint>
 <!-- fixed -->
@@ -195,5 +197,5 @@
   <child link="endeffector_link_1"/>
   <axis xyz="0.0 -1.0 0.0"/>
-  <limit upper="0.698132" lower="-0.698132" effort="100" velocity="100"/>
+  <limit upper="${theta4_max}" lower="${theta4_min}" effort="${effort_max}" velocity="${velocity_max}"/>
 </joint>
 </robot>

Commit message: Adding new URDF of GRASPE

File: ros_ws/src/graspe_description/urdf/graspe.xacro (robot description, xacro)
@@ -1,4 +1,5 @@
 <?xml version="1.0" ?>
 <robot name="graspe" xmlns:xacro="http://www.ros.org/wiki/xacro">
+<!-- include -->
 <xacro:include filename="$(find graspe_description)/urdf/materials.xacro" />
 <xacro:include filename="$(find graspe_description)/urdf/graspe.trans" />
@@ -6,19 +7,9 @@
 <xacro:include filename="$(find graspe_description)/urdf/graspe_joints_limits.xacro" />
 <xacro:include filename="$(find graspe_description)/urdf/graspe_gazebo_control.xacro" />
-<!-- Theta1 -->
-<xacro:property name="ajuste1" value="0.04"/>
-<xacro:property name="ajuste2" value="0.083"/>
-<xacro:property name="ajuste3" value="0.0405"/>
-<xacro:property name="ajuste4" value="0.128004"/>
-<xacro:property name="ajuste5" value="0.05"/>
-<xacro:property name="ajuste6" value="0.01"/>
-<xacro:property name="ajuste7" value="0.025004"/>
-<xacro:property name="ajuste8" value="${0.2105 + 0.158 - ajuste4 }"/>
-<xacro:property name="ajuste9" value="0.015"/>
 <link name="base_link">
   <inertial>
-    <origin xyz="-3.793254127438435e-18 -3.793254127438435e-18 0.026500000000000003" rpy="0 0 0"/>
-    <mass value="1.1763536611734302"/>
-    <inertia ixx="0.00054" iyy="0.00054" izz="0.000529" ixy="0.0" iyz="0.0" ixz="0.0"/>
+    <origin xyz="0 0 0" rpy="0 0 0"/>
+    <mass value="1.5"/>
+    <inertia ixx="0.002199" iyy="0.003694" izz="0.003711" ixy="7e-06" iyz="0.000147" ixz="-1.3e-05"/>
   </inertial>
   <visual>
@@ -36,166 +27,143 @@
   </collision>
 </link>
-<link name="revolution_link_1">
+<!-- first joint (theta1) -->
+<link name="rot1_link">
   <inertial>
-    <origin xyz="0.0 0.0 0.049999999999999996" rpy="0 0 0"/>
-    <mass value="0.9864600932271952"/>
-    <inertia ixx="0.000921" iyy="0.000921" izz="0.000197" ixy="0.0" iyz="0.0" ixz="0.0"/>
+    <origin xyz="0 0 0" rpy="0 0 0"/>
+    <mass value="1.5"/>
+    <inertia ixx="0.002199" iyy="0.003694" izz="0.003711" ixy="7e-06" iyz="0.000147" ixz="-1.3e-05"/>
   </inertial>
   <visual>
-    <origin xyz="0.0 0.0 -0.053" rpy="0 0 0"/>
+    <origin xyz="0 0 0" rpy="0 0 0"/>
     <geometry>
-      <mesh filename="file://$(find graspe_description)/meshes/revolution_link_1.stl" scale="0.001 0.001 0.001"/>
+      <mesh filename="file://$(find graspe_description)/meshes/rot1.stl" scale="0.001 0.001 0.001"/>
     </geometry>
     <material name="silver"/>
   </visual>
   <collision>
-    <origin xyz="0.0 0.0 -0.053" rpy="0 0 0"/>
+    <origin xyz="0 0 0" rpy="0 0 0"/>
     <geometry>
-      <mesh filename="file://$(find graspe_description)/meshes/revolution_link_1.stl" scale="0.001 0.001 0.001"/>
+      <mesh filename="file://$(find graspe_description)/meshes/rot1.stl" scale="0.001 0.001 0.001"/>
     </geometry>
   </collision>
 </link>
 <joint name="theta1" type="revolute">
-  <origin xyz="0.0 0.0 0.053" rpy="0 0 0"/>
+  <origin xyz="0.0 0.0 0.08" rpy="0.0 0.0 0.0"/>
   <parent link="base_link"/>
-  <child link="revolution_link_1"/>
+  <child link="rot1_link"/>
   <axis xyz="0.0 0.0 1.0"/>
-  <limit upper="${theta1_max}" lower="${theta1_min}" effort="${effort_max}" velocity="${velocity_max}"/>
+  <limit lower="${theta1_min}" upper="${theta1_max}" effort="${effort_max}" velocity="${velocity_max}"/>
 </joint>
-<!-- Fixed jointJoint -->
-<link name="fixed_link_1">
+<!-- second joint (theta2) -->
+<link name="rot2_link">
   <inertial>
-    <origin xyz="0.0 -0.017499999999999998 ${-0.04083760550324669 + ajuste1}" rpy="0 0 0"/>
-    <mass value="0.1984169956244406"/>
-    <inertia ixx="5e-05" iyy="1.6e-05" izz="4.9e-05" ixy="0.0" iyz="0.0" ixz="0.0"/>
+    <origin xyz="0 0 0" rpy="0 0 1.5707"/>
+    <mass value="1.5"/>
+    <inertia ixx="0.002199" iyy="0.003694" izz="0.003711" ixy="7e-06" iyz="0.000147" ixz="-1.3e-05"/>
   </inertial>
   <visual>
-    <origin xyz="-0.0 0.0 ${-0.206 + ajuste1}" rpy="0 0 0"/>
+    <origin xyz="0 0 0" rpy="0 0 1.5707"/>
     <geometry>
-      <mesh filename="file://$(find graspe_description)/meshes/fixed_link_1.stl" scale="0.001 0.001 0.001"/>
+      <mesh filename="file://$(find graspe_description)/meshes/rot2.stl" scale="0.001 0.001 0.001"/>
     </geometry>
     <material name="silver"/>
   </visual>
   <collision>
-    <origin xyz="-0.0 0.0 ${-0.206 + ajuste1}" rpy="0 0 0"/>
+    <origin xyz="0 0 0" rpy="0 0 1.5707"/>
     <geometry>
-      <mesh filename="file://$(find graspe_description)/meshes/fixed_link_1.stl" scale="0.001 0.001 0.001"/>
+      <mesh filename="file://$(find graspe_description)/meshes/rot2.stl" scale="0.001 0.001 0.001"/>
     </geometry>
   </collision>
 </link>
-<joint name="rigid1" type="fixed">
-  <origin xyz="0.0 0.0 ${0.153 - ajuste1}" rpy="0 0 0"/>
-  <parent link="revolution_link_1"/>
-  <child link="fixed_link_1"/>
+<joint name="theta2" type="revolute">
+  <origin xyz="0.0 0.0 0.119" rpy="0.0 0.0 0.0"/>
+  <parent link="rot1_link"/>
+  <child link="rot2_link"/>
+  <axis xyz="0.0 1.0 0.0"/>
+  <limit lower="${theta2_min}" upper="${theta2_max}" effort="${effort_max}" velocity="${velocity_max}"/>
 </joint>
-<!-- Theta2 -->
-<link name="revolution2_link_1">
+<!-- prismatic joint (d3) -->
+<link name="prismatic3_link">
   <inertial>
-    <origin xyz="4.126627129485931e-08 ${0.12800435621809492 - ajuste4} ${0.0647561892724049 - ajuste2 + ajuste3}" rpy="0 0 0"/>
-    <mass value="0.06955361957457033"/>
-    <inertia ixx="1.6e-05" iyy="1.8e-05" izz="1.8e-05" ixy="-0.0" iyz="0.0" ixz="0.0"/>
+    <origin xyz="0 0 0" rpy="0 0 3.1415"/>
+    <mass value="1.5"/>
+    <inertia ixx="0.002199" iyy="0.003694" izz="0.003711" ixy="7e-06" iyz="0.000147" ixz="-1.3e-05"/>
   </inertial>
   <visual>
-    <origin xyz="0.0 ${0.158 - ajuste4} ${-0.123 - ajuste2 + ajuste3}" rpy="0 0 0"/>
+    <origin xyz="0 0 0" rpy="0 0 3.1415"/>
     <geometry>
-      <mesh filename="file://$(find graspe_description)/meshes/revolution2_link_1.stl" scale="0.001 0.001 0.001"/>
+      <mesh filename="file://$(find graspe_description)/meshes/prismatic3.stl" scale="0.001 0.001 0.001"/>
     </geometry>
     <material name="silver"/>
   </visual>
   <collision>
-    <origin xyz="0.0 ${0.158 - ajuste4} ${-0.123 - ajuste2 + ajuste3}" rpy="0 0 0"/>
+    <origin xyz="0 0 0" rpy="0 0 3.1415"/>
     <geometry>
-      <mesh filename="file://$(find graspe_description)/meshes/revolution2_link_1.stl" scale="0.001 0.001 0.001"/>
+      <mesh filename="file://$(find graspe_description)/meshes/prismatic3.stl" scale="0.001 0.001 0.001"/>
     </geometry>
   </collision>
 </link>
-<joint name="theta2" type="revolute">
-  <origin xyz="-0.0 ${-0.158 + ajuste4} ${-0.083 + ajuste2}" rpy="0 0 0"/>
-  <parent link="fixed_link_1"/>
-  <child link="revolution2_link_1"/>
-  <axis xyz="0.0 -1.0 0.0"/>
-  <limit upper="${theta2_max}" lower="${theta2_min}" effort="${effort_max}" velocity="${velocity_max}"/>
+<joint name="d3" type="prismatic">
+  <origin xyz="-0.023 0.0 0.008" rpy="0.0 0.0 0.0"/>
+  <parent link="rot2_link"/>
+  <child link="prismatic3_link"/>
+  <axis xyz="0.0 0.0 1.0"/>
+  <limit lower="${d3_min}" upper="${d3_max}" effort="${effort_max}" velocity="${velocity_max}"/>
 </joint>
-<!-- d3 -->
-<link name="slider_link_1">
+<!-- End effector (theta4) -->
+<link name="rot4_link">
   <inertial>
-    <origin xyz="0.0 3.562180949066851e-07 0.01999999999999999" rpy="0 0 0"/>
-    <mass value="0.22195352097611884"/>
-    <inertia ixx="4.2e-05" iyy="4.2e-05" izz="2.5e-05" ixy="0.0" iyz="0.0" ixz="0.0"/>
+    <origin xyz="0 0 0" rpy="0 1.5707 3.1415"/>
+    <mass value="1.5"/>
+    <inertia ixx="0.002199" iyy="0.003694" izz="0.003711" ixy="7e-06" iyz="0.000147" ixz="-1.3e-05"/>
   </inertial>
   <visual>
-    <origin xyz="-0.0 0.029996 -0.2055" rpy="0 0 0"/>
+    <origin xyz="0 0 0" rpy="0 1.5707 3.1415"/>
     <geometry>
-      <mesh filename="file://$(find graspe_description)/meshes/slider_link_1.stl" scale="0.001 0.001 0.001"/>
+      <mesh filename="file://$(find graspe_description)/meshes/rot4.stl" scale="0.001 0.001 0.001"/>
     </geometry>
     <material name="silver"/>
   </visual>
   <collision>
-    <origin xyz="-0.0 0.029996 -0.2055" rpy="0 0 0"/>
+    <origin xyz="0 0 0" rpy="0 1.5707 3.1415"/>
     <geometry>
-      <mesh filename="file://$(find graspe_description)/meshes/slider_link_1.stl" scale="0.001 0.001 0.001"/>
+      <mesh filename="file://$(find graspe_description)/meshes/rot4.stl" scale="0.001 0.001 0.001"/>
     </geometry>
   </collision>
 </link>
-<joint name="d3" type="prismatic">
-  <origin xyz="0.0 ${0.128004 - ajuste4} ${0.0825 - ajuste5}" rpy="0 0 0"/>
-  <parent link="revolution2_link_1"/>
-  <child link="slider_link_1"/>
+<joint name="theta4" type="revolute">
+  <origin xyz="0.0195 -0.015 0.1605" rpy="1.5707 0.0 0.0"/>
+  <parent link="prismatic3_link"/>
+  <child link="rot4_link"/>
   <axis xyz="0.0 0.0 1.0"/>
-  <limit upper="${d3_max}" lower="${d3_min}" effort="${effort_max}" velocity="${velocity_max}"/>
+  <limit lower="${theta4_min}" upper="${theta4_max}" effort="${effort_max}" velocity="${velocity_max}"/>
 </joint>
-<!-- fixed -->
-<link name="fixed2_link_1">
+<!-- end effector (scissor) -->
+<link name="rot5_link">
   <inertial>
-    <origin xyz="0.0 0.015000356218094904 ${0.00964996017692743 - ajuste6}" rpy="0 0 0"/>
-    <mass value="0.15384250264568528"/>
-    <inertia ixx="5e-05" iyy="8e-06" izz="5e-05" ixy="0.0" iyz="0.0" ixz="0.0"/>
+    <origin xyz="0 0 0.006" rpy="0 0 -3.1415"/>
+    <mass value="1.5"/>
+    <inertia ixx="0.002199" iyy="0.003694" izz="0.003711" ixy="7e-06" iyz="0.000147" ixz="-1.3e-05"/>
   </inertial>
   <visual>
-    <origin xyz="0.0 0.029996 ${-0.2455 - ajuste6}" rpy="0 0 0"/>
+    <origin xyz="0 0 0.006" rpy="0 0 -3.1415"/>
     <geometry>
-      <mesh filename="file://$(find graspe_description)/meshes/fixed2_link_1.stl" scale="0.001 0.001 0.001"/>
+      <mesh filename="file://$(find graspe_description)/meshes/rot5.stl" scale="0.001 0.001 0.001"/>
     </geometry>
     <material name="silver"/>
   </visual>
   <collision>
-    <origin xyz="0.0 0.029996 ${-0.2455 - ajuste6}" rpy="0 0 0"/>
+    <origin xyz="0 0 0.006" rpy="0 0 -3.1415"/>
     <geometry>
-      <mesh filename="file://$(find graspe_description)/meshes/fixed2_link_1.stl" scale="0.001 0.001 0.001"/>
+      <mesh filename="file://$(find graspe_description)/meshes/rot5.stl" scale="0.001 0.001 0.001"/>
     </geometry>
   </collision>
 </link>
-<joint name="rigid2" type="fixed">
-  <origin xyz="-0.0 0.0 ${0.04 + ajuste6}" rpy="0 0 0"/>
-  <parent link="slider_link_1"/>
-  <child link="fixed2_link_1"/>
-</joint>
-<!-- Theta4 -->
-<link name="endeffector_link_1">
-  <inertial>
-    <origin xyz="-3.206969956259798e-10 ${0.24049635982298995 - ajuste8} ${-0.002508226805447933 + ajuste9}" rpy="0 0 0"/>
-    <mass value="0.1076530467419571"/>
-    <inertia ixx="1.1e-05" iyy="1.3e-05" izz="1.8e-05" ixy="-0.0" iyz="-0.0" ixz="-0.0"/>
-  </inertial>
-  <visual>
-    <origin xyz="-0.0 ${0.240496 - ajuste8} ${-0.270504 + ajuste9}" rpy="0 0 0"/>
-    <geometry>
-      <mesh filename="file://$(find graspe_description)/meshes/endeffector_link_1.stl" scale="0.001 0.001 0.001"/>
-    </geometry>
-    <material name="silver"/>
-  </visual>
-  <collision>
-    <origin xyz="-0.0 ${0.240496 - ajuste8} ${-0.270504 + ajuste9}" rpy="0 0 0"/>
-    <geometry>
-      <mesh filename="file://$(find graspe_description)/meshes/endeffector_link_1.stl" scale="0.001 0.001 0.001"/>
-    </geometry>
-  </collision>
-</link>
-<joint name="theta4" type="revolute">
-  <origin xyz="0.0 ${-0.2105 + ajuste8} ${0.025004 - ajuste7}" rpy="0 0 0"/>
-  <parent link="fixed2_link_1"/>
-  <child link="endeffector_link_1"/>
-  <axis xyz="0.0 -1.0 0.0"/>
-  <limit upper="${theta4_max}" lower="${theta4_min}" effort="${effort_max}" velocity="${velocity_max}"/>
+<joint name="scissor" type="revolute">
+  <origin xyz="0.0 0.06715 -0.02" rpy="0.0 -1.5707 0.0"/>
+  <parent link="rot4_link"/>
+  <child link="rot5_link"/>
+  <axis xyz="0.0 0.0 1.0"/>
+  <limit lower="${scissor_min}" upper="${scissor_max}" effort="${effort_max}" velocity="${velocity_max}"/>
 </joint>
 </robot>

File: ros_ws/src/graspe_description/urdf/graspe_gazebo_control.xacro (robot description, xacro)
@@ -37,5 +37,5 @@
             </command_interface>
             <state_interface name="position">
-                <param name="initial_value">-0.026</param>
+                <param name="initial_value">0.0</param>
             </state_interface>
             <state_interface name="velocity"/>
@@ -54,4 +54,16 @@
             <state_interface name="effort"/>
         </joint>
+        <!-- scissor -->
+        <joint name="scissor">
+            <command_interface name="position">
+                <param name="min">${scissor_min}</param>
+                <param name="max">${scissor_max}</param>
+            </command_interface>
+            <state_interface name="position">
+                <param name="initial_value">0.0</param>
+            </state_interface>
+            <state_interface name="velocity"/>
+            <state_interface name="effort"/>
+        </joint>
     </ros2_control>
 </robot>

File: ros_ws/src/graspe_description/urdf/graspe_joints_limits.xacro (robot description, xacro)
@@ -3,10 +3,12 @@
     <xacro:property name="theta1_max" value="3.1415"/>
     <xacro:property name="theta1_min" value="${-theta1_max}"/>
-    <xacro:property name="theta2_max" value="2.61799"/>
+    <xacro:property name="theta2_max" value="3.1415"/>
     <xacro:property name="theta2_min" value="${-theta2_max}"/>
     <xacro:property name="d3_max" value="0.00"/>
-    <xacro:property name="d3_min" value="-0.026"/>
-    <xacro:property name="theta4_max" value="1.5708"/>
+    <xacro:property name="d3_min" value="-0.070"/>
+    <xacro:property name="theta4_max" value="3.1415"/>
     <xacro:property name="theta4_min" value="${-theta4_max}"/>
+    <xacro:property name="scissor_max" value="0.35"/>
+    <xacro:property name="scissor_min" value="-0.49"/>
     <xacro:property name="velocity_max" value="10.0"/>
     <xacro:property name="effort_max" value="10.0"/>

Commit message: Added camera on end effector, todo: depth, seg, placement

File: ros_ws/src/graspe_description/urdf/graspe.xacro (robot description, xacro)
@@ -7,8 +7,9 @@
 <xacro:include filename="$(find graspe_description)/urdf/graspe_joints_limits.xacro" />
 <xacro:include filename="$(find graspe_description)/urdf/graspe_gazebo_control.xacro" />
+<link name="world" />
 <link name="base_link">
   <inertial>
     <origin xyz="0 0 0" rpy="0 0 0"/>
-    <mass value="1.5"/>
+    <mass value="10.0"/>
     <inertia ixx="0.002199" iyy="0.003694" izz="0.003711" ixy="7e-06" iyz="0.000147" ixz="-1.3e-05"/>
   </inertial>
@@ -27,9 +28,15 @@
   </collision>
 </link>
+<!-- fixing base_link-->
+<joint name="world_joint" type="fixed">
+    <parent link="world" />
+    <child link = "base_link" />
+    <origin xyz="0.0 0.0 0.0" rpy="0.0 0.0 0.0" />
+  </joint>
 <!-- first joint (theta1) -->
 <link name="rot1_link">
   <inertial>
     <origin xyz="0 0 0" rpy="0 0 0"/>
-    <mass value="1.5"/>
+    <mass value="0.150"/>
     <inertia ixx="0.002199" iyy="0.003694" izz="0.003711" ixy="7e-06" iyz="0.000147" ixz="-1.3e-05"/>
   </inertial>
@@ -59,5 +66,5 @@
   <inertial>
     <origin xyz="0 0 0" rpy="0 0 1.5707"/>
-    <mass value="1.5"/>
+    <mass value="0.150"/>
     <inertia ixx="0.002199" iyy="0.003694" izz="0.003711" ixy="7e-06" iyz="0.000147" ixz="-1.3e-05"/>
   </inertial>
@@ -87,5 +94,5 @@
   <inertial>
     <origin xyz="0 0 0" rpy="0 0 3.1415"/>
-    <mass value="1.5"/>
+    <mass value="0.150"/>
     <inertia ixx="0.002199" iyy="0.003694" izz="0.003711" ixy="7e-06" iyz="0.000147" ixz="-1.3e-05"/>
   </inertial>
@@ -115,5 +122,5 @@
   <inertial>
     <origin xyz="0 0 0" rpy="0 1.5707 3.1415"/>
-    <mass value="1.5"/>
+    <mass value="0.150"/>
     <inertia ixx="0.002199" iyy="0.003694" izz="0.003711" ixy="7e-06" iyz="0.000147" ixz="-1.3e-05"/>
   </inertial>
@@ -143,5 +150,5 @@
   <inertial>
     <origin xyz="0 0 0.006" rpy="0 0 -3.1415"/>
-    <mass value="1.5"/>
+    <mass value="0.150"/>
     <inertia ixx="0.002199" iyy="0.003694" izz="0.003711" ixy="7e-06" iyz="0.000147" ixz="-1.3e-05"/>
   </inertial>
@@ -167,3 +174,38 @@
   <limit lower="${scissor_min}" upper="${scissor_max}" effort="${effort_max}" velocity="${velocity_max}"/>
 </joint>
+<link name="camera_link"></link>
+<joint name="camera_joint" type="fixed">
+    <parent link="rot4_link"/>
+    <child link="camera_link"/>
+    <origin xyz="0.03 0.05 -0.02" rpy="-1.5707 0.0 1.5707"/>
+</joint>
+<joint name="camera_optical_joint" type="fixed">
+    <origin xyz="0 0 0" rpy="-1.5707 0 -1.5707" />
+    <parent link="camera_link" />
+    <child link="camera_link_optical" />
+</joint>
+<link name="camera_link_optical"></link>
+<gazebo reference="camera_link">
+    <sensor name="camera" type="camera">
+            <pose> 0 0 0 0 0 0 </pose>
+            <visualize>true</visualize>
+            <update_rate>30</update_rate>
+            <camera>
+                <horizontal_fov>1.089</horizontal_fov>
+                <image>
+                    <format>R8G8B8</format>
+                    <width>640</width>
+                    <height>480</height>
+                </image>
+                <clip>
+                    <near>0.05</near>
+                    <far>8.0</far>
+                </clip>
+            </camera>
+            <plugin name="camera_controller" filename="libgazebo_ros_camera.so">
+                <frame_name>camera_link_optical</frame_name>
+                <alwaysOn>true</alwaysOn>
+            </plugin>
+        </sensor>
+</gazebo>
 </robot>

File: ros_ws/src/graspe_description/urdf/graspe_joints_limits.xacro (robot description, xacro)
@@ -12,4 +12,4 @@
     <xacro:property name="scissor_min" value="-0.49"/>
     <xacro:property name="velocity_max" value="10.0"/>
-    <xacro:property name="effort_max" value="10.0"/>
+    <xacro:property name="effort_max" value="2.0"/>
 </robot>

Commit message: MInor changes to rviz and urdf

File: ros_ws/src/graspe_description/urdf/graspe.xacro (robot description, xacro)
@@ -84,5 +84,5 @@
 </link>
 <joint name="theta2" type="revolute">
-  <origin xyz="0.0 0.0 0.119" rpy="0.0 0.0 0.0"/>
+  <origin xyz="0.0 0.0 0.122" rpy="0.0 0.0 0.0"/>
   <parent link="rot1_link"/>
   <child link="rot2_link"/>

File: ros_ws/src/graspe_description/urdf/graspe_joints_limits.xacro (robot description, xacro)
@@ -3,10 +3,10 @@
     <xacro:property name="theta1_max" value="3.1415"/>
     <xacro:property name="theta1_min" value="${-theta1_max}"/>
-    <xacro:property name="theta2_max" value="3.1415"/>
-    <xacro:property name="theta2_min" value="${-theta2_max}"/>
+    <xacro:property name="theta2_max" value="1.5707"/>
+    <xacro:property name="theta2_min" value="0.764"/>
     <xacro:property name="d3_max" value="0.00"/>
     <xacro:property name="d3_min" value="-0.070"/>
-    <xacro:property name="theta4_max" value="3.1415"/>
-    <xacro:property name="theta4_min" value="${-theta4_max}"/>
+    <xacro:property name="theta4_max" value="0.221"/>
+    <xacro:property name="theta4_min" value="-0.662"/>
     <xacro:property name="scissor_max" value="0.35"/>
     <xacro:property name="scissor_min" value="-0.49"/>
