Commit message: Inicial Graspe URDF bugs fixed

File: ros_ws/install/graspeurdf_description/share/graspeurdf_description/urdf/graspeurdf.xacro (robot description, xacro)
@@ -31,5 +31,5 @@
   </inertial>
   <visual>
-    <origin xyz="0.0 0.029996 -0.2455" rpy="0 0 0"/>
+    <origin xyz="0.0 0.029996 -0.255" rpy="0 0 0"/>
     <geometry>
       <mesh filename="file://$(find graspeurdf_description)/meshes/rotacionalpequeno_1.stl" scale="0.001 0.001 0.001"/>
@@ -51,5 +51,5 @@
   </inertial>
   <visual>
-    <origin xyz="-0.0 0.240496 -0.270504" rpy="0 0 0"/>
+    <origin xyz="-0.0 0.0 -0.255" rpy="0 0 0"/>
     <geometry>
       <mesh filename="file://$(find graspeurdf_description)/meshes/endfactor_1.stl" scale="0.001 0.001 0.001"/>
@@ -91,5 +91,5 @@
   </inertial>
   <visual>
-    <origin xyz="-0.0 0.0 -0.206" rpy="0 0 0"/>
+    <origin xyz="-0.0 0.0 -0.165" rpy="0 0 0"/>
     <geometry>
       <mesh filename="file://$(find graspeurdf_description)/meshes/rotacionalgrande_1.stl" scale="0.001 0.001 0.001"/>
@@ -111,5 +111,5 @@
   </inertial>
   <visual>
-    <origin xyz="0.0 0.158 -0.123" rpy="0 0 0"/>
+    <origin xyz="0.0 0.03 -0.17" rpy="0 0 0"/>
     <geometry>
       <mesh filename="file://$(find graspeurdf_description)/meshes/prismatica_1.stl" scale="0.001 0.001 0.001"/>
@@ -145,16 +145,10 @@
 </link>
 <joint name="Rigid 5" type="fixed">
-  <origin xyz="-0.0 0.0 0.04" rpy="0 0 0"/>
+  <origin xyz="-0.0 0.0 0.05" rpy="0 0 0"/>
   <parent link="linkpequeno_1"/>
   <child link="rotacionalpequeno_1"/>
 </joint>
-<joint name="endfactor" type="revolute">
-  <origin xyz="0.0 -0.2105 0.025004" rpy="0 0 0"/>
-  <parent link="rotacionalpequeno_1"/>
-  <child link="endfactor_1"/>
-  <axis xyz="0.0 -1.0 0.0"/>
-  <limit upper="0.698132" lower="-0.698132" effort="100" velocity="100"/>
-</joint>
-<joint name="Revolute 7" type="continuous">
+<!-- Theta1 -->
+<joint name="theta1" type="continuous">
   <origin xyz="0.0 0.0 0.053" rpy="0 0 0"/>
   <parent link="base_link"/>
@@ -163,17 +157,19 @@
 </joint>
 <joint name="Rigid 8" type="fixed">
-  <origin xyz="0.0 0.0 0.153" rpy="0 0 0"/>
+  <origin xyz="0.0 0.0 0.112" rpy="0 0 0"/>
   <parent link="linkgrande_1"/>
   <child link="rotacionalgrande_1"/>
 </joint>
-<joint name="Revolute 9" type="revolute">
-  <origin xyz="-0.0 -0.158 -0.083" rpy="0 0 0"/>
+<!-- theta2 -->
+<joint name="theta2" type="revolute">
+  <origin xyz="-0.0 -0.03 0.0" rpy="0 0 0"/>
   <parent link="rotacionalgrande_1"/>
   <child link="prismatica_1"/>
   <axis xyz="0.0 -1.0 0.0"/>
-  <limit upper="0.785398" lower="-0.785398" effort="100" velocity="100"/>
+  <limit upper="3.1415" lower="-3.1415" effort="100" velocity="100"/>
 </joint>
-<joint name="prismatica1" type="prismatic">
-  <origin xyz="0.0 0.128004 0.0825" rpy="0 0 0"/>
+<!-- Prismatic d3 -->
+<joint name="d3" type="prismatic">
+  <origin xyz="0.0 0.0 0.0825" rpy="0 0 0"/>
   <parent link="prismatica_1"/>
   <child link="linkpequeno_1"/>
@@ -181,3 +177,11 @@
   <limit lower="0.0" upper="0.1" effort="50" velocity="0.2"/>
 </joint>
+<!-- theta4 end effector -->
+<joint name="theta4" type="revolute">
+  <origin xyz="0.0 0.03 0.0" rpy="0 0 0"/>
+  <parent link="rotacionalpequeno_1"/>
+  <child link="endfactor_1"/>
+  <axis xyz="0.0 -1.0 0.0"/>
+  <limit upper="0.698132" lower="-0.698132" effort="100" velocity="100"/>
+</joint>
 </robot>
